File: GD32F470.brd (EAGLE design)
At the start: 81 x 82.5 mm, 103 parts, among them CN1 CLOCK-1-2, CN2 CLOCK-3-4, CN3 CLOCK-5-6, CN4 CLOCK-7-8, J1 BOOT0, J2 I2C+INT, J3 USB_A_SMT_FEMALE, J4 RJ45, J5 RJ45, J6 RJ45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

Commit message: Replace USB-A footprint
Swap SparkFun USB-A footprint for a local GD32F USB-A (new library/packages and 3D package), update footprint URNs/library_version for multiple parts (1X03, SO08-EIAJ, 1X05, etc.), and adjust board element attributes (J1, U3, U1) and coordinates. Reroute and reconnect USB nets (VBUS, D+, D-, SHLD) to match the new footprint, add a SHLD signal, and tidy related wire widths/paths. Add new schematic GD32F470.sch and update binary BOM/CPL and Gerber outputs.
Parts:
- J1: value BOOT0 -> 455-1750-1-ND
- J3: device SparkFun-Connectors:USB-A-S-SILK-FEMALE -> GD32F:USB-A
- U3: value W25Q128JVSIQ -> 25F32006WSOI
- moved J3 3.49 mm to (77.8, 36.5)
- moved R6 0.95 mm to (63.2, 35.6)
- moved R7 0.32 mm to (63.2, 37.5)
Connections:
- net N$49 renamed SHLD
Routing:
- net SHLD: track 18.7 -> 25.9 mm
- net +5V: track 100.2 -> 103.7 mm
- net N$47: track 3.51 -> 6.91 mm
- net N$20: track 3.81 -> 6.91 mm
- net PA11: track 30.5 -> 31.9 mm
